File: CH559Pico.kicad_pcb (KiCad board)
At the start: 2 copper layers, 21 x 50.8 mm, 20 parts, among them CN1 CON_USB-C-16, J1 Conn_01x20, J2 Conn_01x20, Q1 TR_NMOS_IRLML6344, SW1 SW_Push, SW2 SW_Push, U1 MCU_CH559L

Commit message: update for v2
Parts:
- removed R3: 10k, Resistor_SMD:R_0603_1608Metric
- added J3: Conn_01x01, akita:Pad_SMD1.6mm, B.Cu at (17.8, 25.4)
- added J4: Conn_01x01, akita:Pad_SMD1.6mm, B.Cu at (17.8, 27.9)
- SW1, SW2: footprint Button_Switch_SMD:SW_SPST_PTS810 -> Button_Switch_SMD:SW_Push_SPST_NO_Alps_SKRK
- moved CN1 0.21 mm to (10.5, 5.93)
Connections:
- J2 pad 10: unconnected-(J2-Pad10) -> /P4.7
- J2 pad 17: unconnected-(J2-Pad17) -> /P4.6
- SW2 pad 1: Net-(R3-Pad1) -> /P4.6
- SW2 pad 2: +3V3 -> GND
Routing:
- net /P4.6: track 11.9 -> 28.8 mm
- net Net-(R3-Pad1): track 8.79 -> 0.00 mm
- net +3V3: track 33.0 -> 25.8 mm
- net /P4.7: track 0.00 -> 5.09 mm, vias 0 -> 1
- net +5V: track 45.1 -> 47.7 mm
- net GND: track 154.1 -> 156.4 mm
- net /P2.1: track 8.57 -> 7.81 mm
- added copper zone on B.Cu, net GND
- added copper zone on F.Cu, net GND
Other:
- board text added: "4.6"
- board text added: "4.7"
- board text added: "X4.6"
- board text added: "X4.7"
- board text added: "v2"
