File: CH559Pico.kicad_sch (KiCad schematic)
At the start: 18 parts, among them CN1 CON_USB-C-16, J1 Conn_01x20, J2 Conn_01x20, Q1 TR_NMOS_IRLML6344, SW1 SW_Push, SW2 SW_Push, U1 MCU_CH559L

Commit message: update for v2
Parts:
- removed R3: 10k, Resistor_SMD:R_0603_1608Metric, symbol Device:R
- added J3, J4: Conn_01x01, akita:Pad_SMD1.6mm, symbol Connector_Generic:Conn_01x01
- C1, C2: LCSC (none) -> C14663
- CN1: LCSC (none) -> C165948
- D1: LCSC (none) -> C165982
- D2: LCSC (none) -> C138546
- D3: LCSC (none) -> C190475
- F1: LCSC (none) -> C2982267
- Q1: LCSC (none) -> C20917
- R1, R2: LCSC (none) -> C23186
- R4, R5: LCSC (none) -> C21190
- SW1, SW2: footprint Button_Switch_SMD:SW_SPST_PTS810 -> Button_Switch_SMD:SW_Push_SPST_NO_Alps_SKRK; LCSC (none) -> C2837082
- U1: LCSC (none) -> C150548
Connections:
- net +3V3: no longer SW2.2
- net GND: now also SW2.2
- net P4.6: now also J2.17 (Pin_17), SW2.1, J3.1 (Pin_1)
- net P4.7: now also J2.10 (Pin_10), J4.1 (Pin_1)
- no-connect marks 4 -> 2
